Commit message: Fix avionics box and mast urdf model

File: data/urdf/sherpa_tt.urdf (robot description, URDF)
Before this commit: robot Sherpa_tt, 47 links, 46 joints
Links:
- added link box_base; collision box size=0.355 0.600 0.042; visual box size=0.355 0.600 0.042
- added link loc_cam; collision box size=0.095 0.576 0.1; visual box size=0.095 0.576 0.1
- added link nav_cam; collision box size=0.042 0.38 0.034; visual box size=0.042 0.38 0.034
- link box: geometry collision box size=0.26 0.395 0.39; visual box size=0.26 0.395 0.39
- link mast: geometry collision box size=0.160 0.045 1.118; visual box size=0.160 0.045 1.118
Joints:
- added joint box_to_box_base: type fixed, parent box, child box_base
- added joint mast_to_loc_cam: type fixed, parent mast, child loc_cam
- added joint mast_to_nav_cam: type fixed, parent mast, child nav_cam
