Commit message: Modify urdf files to allow collision detection of the manipulator with itself

File: data/urdf/manipulator.urdf (robot description, URDF)
Before this commit: robot Sherpa_tt, 8 links, 7 joints
Links:
- link arm_link_1: geometry collision cylinder length=0.22 radius=0.08; collision cylinder length=0.45 radius=0.075
- link arm_link_2: geometry collision cylinder length=0.27 radius=0.09; collision cylinder length=0.51 radius=0.04
- link arm_link_3: geometry collision cylinder length=0.4 radius=0.057; visual cylinder length=0.4 radius=0.057
- link arm_link_4: geometry collision cylinder length=0.13 radius=0.059; collision cylinder length=0.2 radius=0.055
- link arm_link_5: geometry collision cylinder length=0.14 radius=0.05; visual cylinder length=0.14 radius=0.05
- link arm_link_6: geometry collision box size=0.17 0.15 0.09; visual box size=0.17 0.15 0.09

File: data/urdf/sherpa_tt.urdf (robot description, URDF)
Before this commit: robot Sherpa_tt, 47 links, 46 joints
Links:
- link box: geometry collision box size=0.15 0.3 0.3; visual box size=0.15 0.3 0.3

Commit message: Improving collision situations detection
Signed-off-by: Ricardo Sanchez <ricardosan@uma.es>

File: data/urdf/manipulator.urdf (robot description, URDF)
Before this commit: robot Sherpa_tt, 8 links, 7 joints
Links:
- link arm_link_1: geometry visual cylinder length=0.22 radius=0.08; visual cylinder length=0.45 radius=0.075

Commit message: Update urdf models
Adapt first joint so it does not collide with the mast; include simple ground collision detection

File: data/urdf/manipulator.urdf (robot description, URDF)
Before this commit: robot Sherpa_tt, 8 links, 7 joints
Links:
- link arm_link_1: geometry collision cylinder length=0.09 radius=0.045; collision cylinder length=0.1 radius=0.045

File: data/urdf/sherpa_tt.urdf (robot description, URDF)
Before this commit: robot Sherpa_tt, 50 links, 49 joints
Links:
- added link ground; collision box size=10 10 0.01; visual box size=10 10 0.01
Joints:
- added joint body_to_ground: type fixed, parent body, child ground

Commit message: Develop arm reachability map computation
Create functions to compute and plot the reachability map; add reachabilityMap; add cartesian space option in collisionPlotter; improve urdf model of the manipulator

File: data/urdf/manipulator.urdf (robot description, URDF)
Before this commit: robot Sherpa_tt, 8 links, 7 joints
Links:
- link arm_link_2: geometry collision cylinder length=0.1 radius=0.05; collision cylinder length=0.148 radius=0.07

Commit message: Improve manipulator urdf collision model
Detail the third link collision model to increase the third joint movement range

File: data/urdf/manipulator.urdf (robot description, URDF)
Before this commit: robot Sherpa_tt, 8 links, 7 joints
Links:
- link arm_link_3: geometry collision cylinder length=0.11 radius=0.057; collision cylinder length=0.29 radius=0.034
