Commit message: Fixing some bugs due to new mast height

File: data/planner/sherpa_tt.urdf (robot description, URDF)
Before this commit: robot Sherpa_tt, 51 links, 50 joints
Links:
- link nav_cam: geometry collision box size=0.3 0.576 0.2; visual box size=0.3 0.576 0.2

Commit message: Field testing 7-8-2020
Signed-off-by: JRicardoSan <ricardosan@uma.es>

File: data/planner/sherpa_tt.urdf (robot description, URDF)
Before this commit: robot Sherpa_tt, 51 links, 50 joints
Links:
- link box: geometry collision box size=0.5 0.395 0.39; visual box size=0.5 0.395 0.39
